Commit message: day0.1

File: assets/urdf/waveshare_5dof.urdf (robot description, URDF)
Before this commit: robot physics, 11 links, 10 joints
Links:
- link base_link: geometry visual mesh filename=package://../meshes/base.stl
- link l1_link: geometry visual mesh filename=package://../meshes/L1.stl
- link l2_link: geometry visual mesh filename=package://../meshes/L2.stl
- link l3_link: geometry visual mesh filename=package://../meshes/L3.stl
- link l4_link: geometry visual mesh filename=package://../meshes/L4.stl
- link l5_1_A_link: geometry visual mesh filename=package://../meshes/L5_1_A.stl
- link l5_1_B_link: geometry visual mesh filename=package://../meshes/L5_1_B.stl
- link l5_2_A_link: geometry visual mesh filename=package://../meshes/L5_2_A.stl
- link l5_2_B_link: geometry visual mesh filename=package://../meshes/L5_2_B.stl
- link l5_3_A_link: geometry visual mesh filename=package://../meshes/L5_3_A.stl
- link l5_3_B_link: geometry visual mesh filename=package://../meshes/L5_3_B.stl
